File: Tactile Browser Hardware/Tactile Browser/Tactile Browser.kicad_pcb (KiCad board)
At the start: 2 copper layers, 79 parts, among them SW1 SW_Push, SW10 SW_Push, SW11 SW_Push, SW12 SW_Push, SW13 SW_Push, SW14 SW_Push, SW15 SW_Push, SW16 SW_Push, SW17 SW_Push, SW18 SW_Push, SW19 SW_Push, SW2 SW_Push, SW20 SW_Push, SW3 SW_Push, SW4 SW_Push, SW5 SW_Push, SW6 SW_Push, SW7 SW_Push, SW8 SW_Push, SW9 SW_Push

Commit message: pcb edits
Parts:
- 12V_supply1: moved to F.Cu
- Driver1, Driver10, Driver2, Driver3, Driver4, Driver5, Driver6, Driver7, Driver8, Driver9: footprint Package_DIP:DIP-24_W15.24mm -> Connector_PinHeader_2.54mm:PinHeader_2x08_P2.54mm_Vertical
- moved 5V_logic_rail1 115.0 mm to (98.2, 174.2)
- moved I2C_bus1 114.7 mm to (108.5, 174.5)
- moved SW9 105.9 mm to (50.0, 60.0)
- moved SW10 95.2 mm to (68.5, 59.5)
- moved SW1 94.7 mm to (49.5, 34.5)
- moved SW13 94.1 mm to (51.0, 110.5)
- moved Driver1 91.3 mm to (56.2, 70.4)
- moved SW2 85.8 mm to (66.5, 34.5)
- moved SW17 81.5 mm to (51.0, 123.5)
- moved SW5 79.1 mm to (49.7, 46.0)
- moved Solenoid5 77.2 mm to (39.7, 47.0)
- moved SW14 75.2 mm to (72.5, 83.5)
- moved SW3 69.7 mm to (91.0, 35.5)
- moved SW6 69.4 mm to (67.7, 45.7)
- moved Solenoid9 66.0 mm to (40.0, 61.0)
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Other:
- board outline added: 100.5 x 100.5 mm

Commit message: update
Parts:
- Driver1, Driver10, Driver2, Driver3, Driver4, Driver5, Driver6, Driver7, Driver8, Driver9: footprint Connector_PinHeader_2.54mm:PinHeader_2x08_P2.54mm_Vertical -> TB6612FNG_THT:TB6612FNG_DualPinHeader_1x8x2_P2.54mm_Row15.24mm_THT
- moved A1 132.5 mm to (39.8, 72.1), turned to 0 degrees
- moved 12V_supply1 123.4 mm to (131.0, 61.0), turned to 90 degrees
- moved Driver10 122.8 mm to (133.7, 31.6)
- moved SW8 114.2 mm to (52.5, 146.0)
- moved 5V_logic_rail1 108.7 mm to (131.0, 70.5), turned to 90 degrees
- moved SW7 107.3 mm to (43.5, 147.0), turned to 180 degrees
- moved SW4 106.8 mm to (41.5, 113.5), turned to 90 degrees
- moved I2C_bus1 98.1 mm to (131.0, 79.0), turned to 90 degrees
- moved Solenoid4 97.6 mm to (50.0, 117.5)
- moved SW6 92.0 mm to (42.0, 134.0), turned to 90 degrees
- moved Driver4 90.5 mm to (74.7, 77.6)
- moved SW9 88.4 mm to (64.2, 147.2)
- moved SW10 87.8 mm to (76.0, 147.0)
- moved Solenoid7 86.7 mm to (65.0, 136.5)
- moved Driver5 86.7 mm to (95.2, 77.5)
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Other:
- board size 100.5 x 100.5 mm -> 100.5 x 125 mm
