File: Tactile Browser Hardware/Tactile Browser v2/_autosave-Tactile Browser.kicad_pcb (KiCad board)
At the start: 4 copper layers, 74.2 x 113.2 mm, 132 parts, among them SW1 SW_Push, SW10 SW_Push, SW11 SW_Push, SW12 SW_Push, SW13 SW_Push, SW14 SW_Push, SW15 SW_Push, SW16 SW_Push, SW17 SW_Push, SW18 SW_Push, SW2 SW_Push, SW3 SW_Push, SW4 SW_Push, SW5 SW_Push, SW6 SW_Push, SW7 SW_Push, SW8 SW_Push, SW9 SW_Push

Commit message: more work on pcb
Parts:
- removed the 100uF1 at (139.9, 27.4)
- removed the 100uF2 at (139.9, 30.4)
- moved 100uF4 88.6 mm to (57.8, 66.8)
- moved 100uF3 80.6 mm to (53.0, 66.8)
- moved 1000uf25V2 0.90 mm to (81.3, 49.8), turned to 180 degrees
- moved 1000uf25V3 0.60 mm to (81.3, 61.2), turned to 180 degrees
- renumbered 100nF1 to 100uF1, 100nF2 to 100uF2
Routing:
- net S3_out2: track 6.04 -> 27.4 mm, vias 0 -> 1
- net S4_out1: track 0.00 -> 17.6 mm, vias 0 -> 1
- net S3_in1: track 0.00 -> 16.8 mm
- net S4_out2: track 3.71 -> 17.9 mm
- net S3_in2: track 0.00 -> 12.1 mm
- net GND: track 22.1 -> 34.0 mm
- net PWM: track 7.56 -> 15.5 mm, vias 0 -> 2
- net DATA: track 0.00 -> 4.53 mm, vias 0 -> 1
- net S3_out1: track 13.9 -> 16.3 mm
- net 12V: track 46.8 -> 48.8 mm, vias 4 -> 5
