File: Tactile Browser Hardware/Tactile Browser v2/Tactile Browser.kicad_sch (KiCad schematic)
At the start: 130 parts, among them SW1 SW_Push, SW10 SW_Push, SW11 SW_Push, SW12 SW_Push, SW13 SW_Push, SW14 SW_Push, SW15 SW_Push, SW16 SW_Push, SW17 SW_Push, SW18 SW_Push, SW2 SW_Push, SW3 SW_Push, SW4 SW_Push, SW5 SW_Push, SW6 SW_Push, SW7 SW_Push, SW8 SW_Push, SW9 SW_Push

Commit message: capacitor naming scheme
Parts:
- renumbered C2_100nF1 to 100nF1, 100nF6 to 100nF10, 100nF9 to 100nF11, 100nF8 to 100nF12, 100nF11 to 100nF13, 100nF10 to 100nF14, 100nF13 to 100nF15, 100nF12 to 100nF16, 100nF15 to 100nF17, 100nF14 to 100nF18, 100nF1 to 100nF2, C2_100nF2 to 100nF3, 100nF2 to 100nF4, C2_100nF3 to 100nF5, 100nF3 to 100nF6, 100nF5 to 100nF7, 100nF4 to 100nF8, 100nF7 to 100nF9
Changed lines of the file:
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@@
 		(dnp no)
 		(fields_autoplaced yes)
-		(property "Reference" "100nF1"
+		(property "Reference" "100nF2"
 			(at 356.87 140.97 90)
 			(effects
@@
 			(project ""
 				(path "/2e399075-89ae-469c-893b-1284214b820d"
-					(reference "100nF1")
+					(reference "100nF2")
 					(unit 1)
 				)
@@
 		(on_board yes)
 		(dnp no)
-		(property "Reference" "100nF7"
+		(property "Reference" "100nF9"
 			(at 367.284 331.47 90)
 			(effects
@@
 			(project "Tactile Browser"
 				(path "/2e399075-89ae-469c-893b-1284214b820d"
-					(reference "100nF7")
+					(reference "100nF9")
 					(unit 1)
 				)
@@
 		(on_board yes)
 		(dnp no)
-		(property "Reference" "100nF3"
+		(property "Reference" "100nF6"
 			(at 357.886 232.41 90)
 			(effects
@@
 			(project "Tactile Browser"
 				(path "/2e399075-89ae-469c-893b-1284214b820d"
-					(reference "100nF3")
+					(reference "100nF6")
 					(unit 1)
 				)
@@
 		(dnp no)
 		(fields_autoplaced yes)
-		(property "Reference" "C2_100nF1"
+		(property "Reference" "100nF1"
 			(at 328.93 147.32 90)
 			(effects
@@
 			(project ""
 				(path "/2e399075-89ae-469c-893b-1284214b820d"
-					(reference "C2_100nF1")
+					(reference "100nF1")
 					(unit 1)
 				)
@@
 		(on_board yes)
 		(dnp no)
-		(property "Reference" "100nF13"
+		(property "Reference" "100nF15"
 			(at 105.664 294.64 90)
 			(effects
@@
 			(project "Tactile Browser"
 				(path "/2e399075-89ae-469c-893b-1284214b820d"
-					(reference "100nF13")
+					(reference "100nF15")
 					(unit 1)
 				)
@@
 		(dnp no)
 		(fields_autoplaced yes)
-		(property "Reference" "C2_100nF3"
+		(property "Reference" "100nF5"
 			(at 339.09 238.76 90)
 			(effects
@@
 			(project "Tactile Browser"
 				(path "/2e399075-89ae-469c-893b-1284214b820d"
-					(reference "C2_100nF3")
+					(reference "100nF5")
 					(unit 1)
 				)
@@
 		(on_board yes)
 		(dnp no)
-		(property "Reference" "100nF9"
+		(property "Reference" "100nF11"
 			(at 108.204 185.42 90)
 			(effects
@@
 			(project "Tactile Browser"
 				(path "/2e399075-89ae-469c-893b-1284214b820d"
-					(reference "100nF9")
+					(reference "100nF11")
 					(unit 1)
 				)
@@
 		(on_board yes)
 		(dnp no)
-		(property "Reference" "100nF5"
+		(property "Reference" "100nF7"
 			(at 426.974 246.38 90)
 			(effects
@@
 			(project "Tactile Browser"
 				(path "/2e399075-89ae-469c-893b-1284214b820d"
-					(reference "100nF5")
+					(reference "100nF7")
 					(unit 1)
 				)
@@
 		(dnp no)
 		(fields_autoplaced yes)
-		(property "Reference" "C2_100nF2"
+		(property "Reference" "100nF3"
 			(at 426.72 146.05 90)
 			(effects
@@
 			(project "Tactile Browser"
 				(path "/2e399075-89ae-469c-893b-1284214b820d"
-					(reference "C2_100nF2")
+					(reference "100nF3")
 					(unit 1)
 				)
@@
 		(on_board yes)
 		(dnp no)
-		(property "Reference" "100nF15"
+		(property "Reference" "100nF17"
 			(at 221.234 297.18 90)
 			(effects
@@
 			(project "Tactile Browser"
 				(path "/2e399075-89ae-469c-893b-1284214b820d"
-					(reference "100nF15")
+					(reference "100nF17")
 					(unit 1)
 				)
@@
 		(dnp no)
 		(fields_autoplaced yes)
-		(property "Reference" "100nF2"
+		(property "Reference" "100nF4"
 			(at 450.85 138.43 90)
 			(effects
@@
 			(project "Tactile Browser"
 				(path "/2e399075-89ae-469c-893b-1284214b820d"
-					(reference "100nF2")
+					(reference "100nF4")
 					(unit 1)
 				)
@@
 		(on_board yes)
 		(dnp no)
-		(property "Reference" "100nF4"
+		(property "Reference" "100nF8"
 			(at 446.786 231.14 90)
 			(effects
@@
 			(project "Tactile Browser"
 				(path "/2e399075-89ae-469c-893b-1284214b820d"
-					(reference "100nF4")
+					(reference "100nF8")
 					(unit 1)
 				)
@@
 		(on_board yes)
 		(dnp no)
-		(property "Reference" "100nF10"
+		(property "Reference" "100nF14"
 			(at 227.076 171.45 90)
 			(effects
@@
 			(project "Tactile Browser"
 				(path "/2e399075-89ae-469c-893b-1284214b820d"
-					(reference "100nF10")
+					(reference "100nF14")
 					(unit 1)
 				)
@@
 		(on_board yes)
 		(dnp no)
-		(property "Reference" "100nF8"
+		(property "Reference" "100nF12"
 			(at 128.016 172.72 90)
 			(effects
@@
 			(project "Tactile Browser"
 				(path "/2e399075-89ae-469c-893b-1284214b820d"
-					(reference "100nF8")
+					(reference "100nF12")
 					(unit 1)
 				)
@@
 		(on_board yes)
 		(dnp no)
-		(property "Reference" "100nF11"
+		(property "Reference" "100nF13"
 			(at 207.264 194.31 90)
 			(effects
@@
 			(project "Tactile Browser"
 				(path "/2e399075-89ae-469c-893b-1284214b820d"
-					(reference "100nF11")
+					(reference "100nF13")
 					(unit 1)
 				)
@@
 		(on_board yes)
 		(dnp no)
-		(property "Reference" "100nF12"
+		(property "Reference" "100nF16"
 			(at 125.476 276.86 90)
 			(effects
@@
 			(project "Tactile Browser"
 				(path "/2e399075-89ae-469c-893b-1284214b820d"
-					(reference "100nF12")
+					(reference "100nF16")
 					(unit 1)
 				)
@@
 		(on_board yes)
 		(dnp no)
-		(property "Reference" "100nF6"
+		(property "Reference" "100nF10"
 			(at 387.096 309.88 90)
 			(effects
@@
 			(project "Tactile Browser"
 				(path "/2e399075-89ae-469c-893b-1284214b820d"
-					(reference "100nF6")
+					(reference "100nF10")
 					(unit 1)
 				)
@@
 		(on_board yes)
 		(dnp no)
-		(property "Reference" "100nF14"
+		(property "Reference" "100nF18"
 			(at 241.046 275.59 90)
 			(effects
@@
 			(project "Tactile Browser"
 				(path "/2e399075-89ae-469c-893b-1284214b820d"
-					(reference "100nF14")
+					(reference "100nF18")
 					(unit 1)
 				)

Commit message: schottky diode placement
Parts:
- renumbered 100nF1 to 100uF1, 100nF10 to 100uF10, 100nF11 to 100uF11, 100nF12 to 100uF12, 100nF13 to 100uF13, 100nF14 to 100uF14, 100nF15 to 100uF15, 100nF16 to 100uF16, 100nF17 to 100uF17, 100nF18 to 100uF18, 100nF2 to 100uF2, 100nF3 to 100uF3, 100nF4 to 100uF4, 100nF5 to 100uF5, 100nF6 to 100uF6, 100nF7 to 100uF7, 100nF8 to 100uF8, 100nF9 to 100uF9
Changed lines of the file:
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@@
 		(dnp no)
 		(fields_autoplaced yes)
-		(property "Reference" "100nF2"
+		(property "Reference" "100uF2"
 			(at 356.87 140.97 90)
 			(effects
@@
 			(project ""
 				(path "/2e399075-89ae-469c-893b-1284214b820d"
-					(reference "100nF2")
+					(reference "100uF2")
 					(unit 1)
 				)
@@
 		(on_board yes)
 		(dnp no)
-		(property "Reference" "100nF9"
+		(property "Reference" "100uF9"
 			(at 367.284 331.47 90)
 			(effects
@@
 			(project "Tactile Browser"
 				(path "/2e399075-89ae-469c-893b-1284214b820d"
-					(reference "100nF9")
+					(reference "100uF9")
 					(unit 1)
 				)
@@
 		(on_board yes)
 		(dnp no)
-		(property "Reference" "100nF6"
+		(property "Reference" "100uF6"
 			(at 357.886 232.41 90)
 			(effects
@@
 			(project "Tactile Browser"
 				(path "/2e399075-89ae-469c-893b-1284214b820d"
-					(reference "100nF6")
+					(reference "100uF6")
 					(unit 1)
 				)
@@
 		(dnp no)
 		(fields_autoplaced yes)
-		(property "Reference" "100nF1"
+		(property "Reference" "100uF1"
 			(at 328.93 147.32 90)
 			(effects
@@
 			(project ""
 				(path "/2e399075-89ae-469c-893b-1284214b820d"
-					(reference "100nF1")
+					(reference "100uF1")
 					(unit 1)
 				)
@@
 		(on_board yes)
 		(dnp no)
-		(property "Reference" "100nF15"
+		(property "Reference" "100uF15"
 			(at 105.664 294.64 90)
 			(effects
@@
 			(project "Tactile Browser"
 				(path "/2e399075-89ae-469c-893b-1284214b820d"
-					(reference "100nF15")
+					(reference "100uF15")
 					(unit 1)
 				)
@@
 		(dnp no)
 		(fields_autoplaced yes)
-		(property "Reference" "100nF5"
+		(property "Reference" "100uF5"
 			(at 339.09 238.76 90)
 			(effects
@@
 			(project "Tactile Browser"
 				(path "/2e399075-89ae-469c-893b-1284214b820d"
-					(reference "100nF5")
+					(reference "100uF5")
 					(unit 1)
 				)
@@
 		(on_board yes)
 		(dnp no)
-		(property "Reference" "100nF11"
+		(property "Reference" "100uF11"
 			(at 108.204 185.42 90)
 			(effects
@@
 			(project "Tactile Browser"
 				(path "/2e399075-89ae-469c-893b-1284214b820d"
-					(reference "100nF11")
+					(reference "100uF11")
 					(unit 1)
 				)
@@
 		(on_board yes)
 		(dnp no)
-		(property "Reference" "100nF7"
+		(property "Reference" "100uF7"
 			(at 426.974 246.38 90)
 			(effects
@@
 			(project "Tactile Browser"
 				(path "/2e399075-89ae-469c-893b-1284214b820d"
-					(reference "100nF7")
+					(reference "100uF7")
 					(unit 1)
 				)
@@
 		(dnp no)
 		(fields_autoplaced yes)
-		(property "Reference" "100nF3"
+		(property "Reference" "100uF3"
 			(at 426.72 146.05 90)
 			(effects
@@
 			(project "Tactile Browser"
 				(path "/2e399075-89ae-469c-893b-1284214b820d"
-					(reference "100nF3")
+					(reference "100uF3")
 					(unit 1)
 				)
@@
 		(on_board yes)
 		(dnp no)
-		(property "Reference" "100nF17"
+		(property "Reference" "100uF17"
 			(at 221.234 297.18 90)
 			(effects
@@
 			(project "Tactile Browser"
 				(path "/2e399075-89ae-469c-893b-1284214b820d"
-					(reference "100nF17")
+					(reference "100uF17")
 					(unit 1)
 				)
@@
 		(dnp no)
 		(fields_autoplaced yes)
-		(property "Reference" "100nF4"
+		(property "Reference" "100uF4"
 			(at 450.85 138.43 90)
 			(effects
@@
 			(project "Tactile Browser"
 				(path "/2e399075-89ae-469c-893b-1284214b820d"
-					(reference "100nF4")
+					(reference "100uF4")
 					(unit 1)
 				)
@@
 		(on_board yes)
 		(dnp no)
-		(property "Reference" "100nF8"
+		(property "Reference" "100uF8"
 			(at 446.786 231.14 90)
 			(effects
@@
 			(project "Tactile Browser"
 				(path "/2e399075-89ae-469c-893b-1284214b820d"
-					(reference "100nF8")
+					(reference "100uF8")
 					(unit 1)
 				)
@@
 		(on_board yes)
 		(dnp no)
-		(property "Reference" "100nF14"
+		(property "Reference" "100uF14"
 			(at 227.076 171.45 90)
 			(effects
@@
 			(project "Tactile Browser"
 				(path "/2e399075-89ae-469c-893b-1284214b820d"
-					(reference "100nF14")
+					(reference "100uF14")
 					(unit 1)
 				)
@@
 		(on_board yes)
 		(dnp no)
-		(property "Reference" "100nF12"
+		(property "Reference" "100uF12"
 			(at 128.016 172.72 90)
 			(effects
@@
 			(project "Tactile Browser"
 				(path "/2e399075-89ae-469c-893b-1284214b820d"
-					(reference "100nF12")
+					(reference "100uF12")
 					(unit 1)
 				)
@@
 		(on_board yes)
 		(dnp no)
-		(property "Reference" "100nF13"
+		(property "Reference" "100uF13"
 			(at 207.264 194.31 90)
 			(effects
@@
 			(project "Tactile Browser"
 				(path "/2e399075-89ae-469c-893b-1284214b820d"
-					(reference "100nF13")
+					(reference "100uF13")
 					(unit 1)
 				)
@@
 		(on_board yes)
 		(dnp no)
-		(property "Reference" "100nF16"
+		(property "Reference" "100uF16"
 			(at 125.476 276.86 90)
 			(effects
@@
 			(project "Tactile Browser"
 				(path "/2e399075-89ae-469c-893b-1284214b820d"
-					(reference "100nF16")
+					(reference "100uF16")
 					(unit 1)
 				)
@@
 		(on_board yes)
 		(dnp no)
-		(property "Reference" "100nF10"
+		(property "Reference" "100uF10"
 			(at 387.096 309.88 90)
 			(effects
@@
 			(project "Tactile Browser"
 				(path "/2e399075-89ae-469c-893b-1284214b820d"
-					(reference "100nF10")
+					(reference "100uF10")
 					(unit 1)
 				)
@@
 		(on_board yes)
 		(dnp no)
-		(property "Reference" "100nF18"
+		(property "Reference" "100uF18"
 			(at 241.046 275.59 90)
 			(effects
@@
 			(project "Tactile Browser"
 				(path "/2e399075-89ae-469c-893b-1284214b820d"
-					(reference "100nF18")
+					(reference "100uF18")
 					(unit 1)
 				)

Commit message: PCB almost done!
Connections:
- net S5_out1: now also DS9.2 (A); no longer DS12.2 (A)
- net S5_out2: now also DS10.2 (A); no longer DS11.2 (A)
- net S6_out1: now also DS11.2 (A); no longer DS10.2 (A)
- net S6_out2: now also DS12.2 (A); no longer DS9.2 (A)
Other:
- moved on the sheet: DS10, DS11, DS12, DS9

Commit message: prepped pcb for assembly
Parts:
- renumbered 100uF1 to 1uF1, 100uF10 to 1uF10, 100uF11 to 1uF11, 100uF12 to 1uF12, 100uF13 to 1uF13, 100uF14 to 1uF14, 100uF15 to 1uF15, 100uF16 to 1uF16, 100uF17 to 1uF17, 100uF18 to 1uF18, 100uF2 to 1uF2, 100uF3 to 1uF3, 100uF4 to 1uF4, 100uF5 to 1uF5, 100uF6 to 1uF6, 100uF7 to 1uF7, 100uF8 to 1uF8, 100uF9 to 1uF9
Changed lines of the file:
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@@
 		(dnp no)
 		(fields_autoplaced yes)
-		(property "Reference" "100uF2"
+		(property "Reference" "1uF2"
 			(at 356.87 140.97 90)
 			(effects
@@
 			(project ""
 				(path "/2e399075-89ae-469c-893b-1284214b820d"
-					(reference "100uF2")
+					(reference "1uF2")
 					(unit 1)
 				)
@@
 		(on_board yes)
 		(dnp no)
-		(property "Reference" "100uF9"
+		(property "Reference" "1uF9"
 			(at 367.284 331.47 90)
 			(effects
@@
 			(project "Tactile Browser"
 				(path "/2e399075-89ae-469c-893b-1284214b820d"
-					(reference "100uF9")
+					(reference "1uF9")
 					(unit 1)
 				)
@@
 		(on_board yes)
 		(dnp no)
-		(property "Reference" "100uF6"
+		(property "Reference" "1uF6"
 			(at 357.886 232.41 90)
 			(effects
@@
 			(project "Tactile Browser"
 				(path "/2e399075-89ae-469c-893b-1284214b820d"
-					(reference "100uF6")
+					(reference "1uF6")
 					(unit 1)
 				)
@@
 		(dnp no)
 		(fields_autoplaced yes)
-		(property "Reference" "100uF1"
+		(property "Reference" "1uF1"
 			(at 328.93 147.32 90)
 			(effects
@@
 			(project ""
 				(path "/2e399075-89ae-469c-893b-1284214b820d"
-					(reference "100uF1")
+					(reference "1uF1")
 					(unit 1)
 				)
@@
 		(on_board yes)
 		(dnp no)
-		(property "Reference" "100uF15"
+		(property "Reference" "1uF15"
 			(at 105.664 294.64 90)
 			(effects
@@
 			(project "Tactile Browser"
 				(path "/2e399075-89ae-469c-893b-1284214b820d"
-					(reference "100uF15")
+					(reference "1uF15")
 					(unit 1)
 				)
@@
 		(dnp no)
 		(fields_autoplaced yes)
-		(property "Reference" "100uF5"
+		(property "Reference" "1uF5"
 			(at 339.09 238.76 90)
 			(effects
@@
 			(project "Tactile Browser"
 				(path "/2e399075-89ae-469c-893b-1284214b820d"
-					(reference "100uF5")
+					(reference "1uF5")
 					(unit 1)
 				)
@@
 		(on_board yes)
 		(dnp no)
-		(property "Reference" "100uF11"
+		(property "Reference" "1uF11"
 			(at 108.204 185.42 90)
 			(effects
@@
 			(project "Tactile Browser"
 				(path "/2e399075-89ae-469c-893b-1284214b820d"
-					(reference "100uF11")
+					(reference "1uF11")
 					(unit 1)
 				)
@@
 		(on_board yes)
 		(dnp no)
-		(property "Reference" "100uF7"
+		(property "Reference" "1uF7"
 			(at 426.974 246.38 90)
 			(effects
@@
 			(project "Tactile Browser"
 				(path "/2e399075-89ae-469c-893b-1284214b820d"
-					(reference "100uF7")
+					(reference "1uF7")
 					(unit 1)
 				)
@@
 		(dnp no)
 		(fields_autoplaced yes)
-		(property "Reference" "100uF3"
+		(property "Reference" "1uF3"
 			(at 426.72 146.05 90)
 			(effects
@@
 			(project "Tactile Browser"
 				(path "/2e399075-89ae-469c-893b-1284214b820d"
-					(reference "100uF3")
+					(reference "1uF3")
 					(unit 1)
 				)
@@
 		(on_board yes)
 		(dnp no)
-		(property "Reference" "100uF17"
+		(property "Reference" "1uF17"
 			(at 221.234 297.18 90)
 			(effects
@@
 			(project "Tactile Browser"
 				(path "/2e399075-89ae-469c-893b-1284214b820d"
-					(reference "100uF17")
+					(reference "1uF17")
 					(unit 1)
 				)
@@
 		(dnp no)
 		(fields_autoplaced yes)
-		(property "Reference" "100uF4"
+		(property "Reference" "1uF4"
 			(at 450.85 138.43 90)
 			(effects
@@
 			(project "Tactile Browser"
 				(path "/2e399075-89ae-469c-893b-1284214b820d"
-					(reference "100uF4")
+					(reference "1uF4")
 					(unit 1)
 				)
@@
 		(on_board yes)
 		(dnp no)
-		(property "Reference" "100uF8"
+		(property "Reference" "1uF8"
 			(at 446.786 231.14 90)
 			(effects
@@
 			(project "Tactile Browser"
 				(path "/2e399075-89ae-469c-893b-1284214b820d"
-					(reference "100uF8")
+					(reference "1uF8")
 					(unit 1)
 				)
@@
 		(on_board yes)
 		(dnp no)
-		(property "Reference" "100uF14"
+		(property "Reference" "1uF14"
 			(at 227.076 171.45 90)
 			(effects
@@
 			(project "Tactile Browser"
 				(path "/2e399075-89ae-469c-893b-1284214b820d"
-					(reference "100uF14")
+					(reference "1uF14")
 					(unit 1)
 				)
@@
 		(on_board yes)
 		(dnp no)
-		(property "Reference" "100uF12"
+		(property "Reference" "1uF12"
 			(at 128.016 172.72 90)
 			(effects
@@
 			(project "Tactile Browser"
 				(path "/2e399075-89ae-469c-893b-1284214b820d"
-					(reference "100uF12")
+					(reference "1uF12")
 					(unit 1)
 				)
@@
 		(on_board yes)
 		(dnp no)
-		(property "Reference" "100uF13"
+		(property "Reference" "1uF13"
 			(at 207.264 194.31 90)
 			(effects
@@
 			(project "Tactile Browser"
 				(path "/2e399075-89ae-469c-893b-1284214b820d"
-					(reference "100uF13")
+					(reference "1uF13")
 					(unit 1)
 				)
@@
 		(on_board yes)
 		(dnp no)
-		(property "Reference" "100uF16"
+		(property "Reference" "1uF16"
 			(at 125.476 276.86 90)
 			(effects
@@
 			(project "Tactile Browser"
 				(path "/2e399075-89ae-469c-893b-1284214b820d"
-					(reference "100uF16")
+					(reference "1uF16")
 					(unit 1)
 				)
@@
 		(on_board yes)
 		(dnp no)
-		(property "Reference" "100uF10"
+		(property "Reference" "1uF10"
 			(at 387.096 309.88 90)
 			(effects
@@
 			(project "Tactile Browser"
 				(path "/2e399075-89ae-469c-893b-1284214b820d"
-					(reference "100uF10")
+					(reference "1uF10")
 					(unit 1)
 				)
@@
 		(on_board yes)
 		(dnp no)
-		(property "Reference" "100uF18"
+		(property "Reference" "1uF18"
 			(at 241.046 275.59 90)
 			(effects
@@
 			(project "Tactile Browser"
 				(path "/2e399075-89ae-469c-893b-1284214b820d"
-					(reference "100uF18")
+					(reference "1uF18")
 					(unit 1)
 				)

Commit message: finished footprints (mostly)
Parts:
- 12V_supply1: footprint TerminalBlock_Phoenix:ScrewTerminal_Vertical_1935310 -> TerminalBlock_MetzConnect:TerminalBlock_MetzConnect_Type094_RT03506HBLU_1x06_P5.00mm_Horizontal
Changed lines of the file:
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@@
 			)
 		)
-		(property "Footprint" "TerminalBlock_Phoenix:ScrewTerminal_Vertical_1935310"
+		(property "Footprint" "TerminalBlock_MetzConnect:TerminalBlock_MetzConnect_Type094_RT03506HBLU_1x06_P5.00mm_Horizontal"
 			(at 24.13 24.13 0)
 			(effects
