File: Tactile Browser Hardware/Tactile-Browser-Keycaps/Tactile-Browser-Keycaps.kicad_sch (KiCad schematic)
At the start: 3 parts, among them J1 Conn_01x01_Pin, J2 Conn_01x01_Pin, SW1 SW_Push

Commit message: ketyswitch
Parts:
- removed J1, J2: Conn_01x01_Pin, Connector_PinHeader_2.54mm:PinHeader_1x01_P2.54mm_Horizontal, symbol Connector:Conn_01x01_Pin
- added J1: Conn_01x02_Pin, Connector_JST:JST_PH_B2B-PH-SM4-TB_1x02-1MP_P2.00mm_Vertical, symbol Connector:Conn_01x02_Pin
Connections:
- net at SW1.2: now also J1.2 (Pin_2)
- net at SW1.1: now also J1.1 (Pin_1)
Changed lines of the file:
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@@
 	(wire
 		(pts
-			(xy 71.12 88.9) (xy 77.47 88.9)
+			(xy 87.63 95.25) (xy 83.82 95.25)
 		)
 		(stroke
@@
 	(wire
 		(pts
-			(xy 87.63 88.9) (xy 92.71 88.9)
+			(xy 77.47 95.25) (xy 81.28 95.25)
+		)
+		(stroke
+			(width 0)
+			(type default)
+		)
+	)
+	(wire
+		(pts
+			(xy 77.47 88.9) (xy 77.47 95.25)
+		)
+		(stroke
+			(width 0)
+			(type default)
+		)
+	)
+	(wire
+		(pts
+			(xy 87.63 88.9) (xy 87.63 95.25)
 		)
 		(stroke
@@
 	)
 	(symbol
-		(lib_id "Connector:Conn_01x01_Pin")
-		(at 97.79 88.9 180)
+		(lib_id "Connector:Conn_01x02_Pin")
+		(at 81.28 100.33 90)
 		(unit 1)
 		(exclude_from_sim no)
@@
 		(fields_autoplaced yes)
 		(property "Reference" "J1"
-			(at 97.155 83.82 0)
+			(at 85.09 98.4249 90)
 			(effects
 				(font
 					(size 1.27 1.27)
 				)
+				(justify right)
 			)
 		)
-		(property "Value" "Conn_01x01_Pin"
-			(at 97.155 86.36 0)
+		(property "Value" "Conn_01x02_Pin"
+			(at 85.09 100.9649 90)
 			(effects
 				(font
 					(size 1.27 1.27)
 				)
+				(justify right)
 			)
 		)
-		(property "Footprint" "Connector_PinHeader_2.54mm:PinHeader_1x01_P2.54mm_Horizontal"
-			(at 97.79 88.9 0)
+		(property "Footprint" "Connector_JST:JST_PH_B2B-PH-SM4-TB_1x02-1MP_P2.00mm_Vertical"
+			(at 81.28 100.33 0)
 			(effects
 				(font
@@
 		)
 		(property "Datasheet" "~"
-			(at 97.79 88.9 0)
+			(at 81.28 100.33 0)
 			(effects
 				(font
@@
 			)
 		)
-		(property "Description" "Generic connector, single row, 01x01, script generated"
-			(at 97.79 88.9 0)
+		(property "Description" "Generic connector, single row, 01x02, script generated"
+			(at 81.28 100.33 0)
 			(effects
 				(font
@@
 		(pin "1"
 		)
+		(pin "2"
+		)
 		(instances
 			(project ""
@@
 					(unit 1)
 				)
-			)
-		)
-	)
-	(symbol
-		(lib_id "Connector:Conn_01x01_Pin")
-		(at 66.04 88.9 0)
-		(unit 1)
-		(exclude_from_sim no)
-		(in_bom yes)
-		(on_board yes)
-		(dnp no)
-		(fields_autoplaced yes)
-		(property "Reference" "J2"
-			(at 66.675 83.82 0)
-			(effects
-				(font
-					(size 1.27 1.27)
-				)
-			)
-		)
-		(property "Value" "Conn_01x01_Pin"
-			(at 66.675 86.36 0)
-			(effects
-				(font
-					(size 1.27 1.27)
-				)
-			)
-		)
-		(property "Footprint" "Connector_PinHeader_2.54mm:PinHeader_1x01_P2.54mm_Horizontal"
-			(at 66.04 88.9 0)
-			(effects
-				(font
-					(size 1.27 1.27)
-				)
-				(hide yes)
-			)
-		)
-		(property "Datasheet" "~"
-			(at 66.04 88.9 0)
-			(effects
-				(font
-					(size 1.27 1.27)
-				)
-				(hide yes)
-			)
-		)
-		(property "Description" "Generic connector, single row, 01x01, script generated"
-			(at 66.04 88.9 0)
-			(effects
-				(font
-					(size 1.27 1.27)
-				)
-				(hide yes)
-			)
-		)
-		(pin "1"
-		)
-		(instances
-			(project ""
-				(path "/2b2b64cd-7c3e-4aae-9375-9f7d6b1a636c"
-					(reference "J2")
-					(unit 1)
-				)
