File: Tactile Browser Hardware/Sidebar/Sidebar.kicad_pcb (KiCad board)
At the start: 2 copper layers, 237.5 x 25 mm, 43 parts, among them J1 Conn_01x02_Pin, J2 Conn_01x02_Pin, J3 Barrel_Jack_Switch, J4 Conn_01x02_Pin, Q1 PMOS, SW10 SW_Push, SW11 SW_Push, SW12 SW_Push, SW6 SW_Push, SW7 SW_Push, SW8 SW_Push, SW9 SW_Push

Commit message: Module prototype
I still need to upload the 3d files for the casings I made, but the main thing is over the past few months I've ordered and soldered all the pcbs and they are all working!! I should've uploaded more changes to github
Parts:
- renumbered 100kR1 to 100k, 1kR1 to 1k
Changed lines of the file:
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@@
 		(descr "Resistor SMD 0805 (2012 Metric), square (rectangular) end terminal, IPC-7351 nominal, (Body size source: IPC-SM-782 page 72, https://www.pcb-3d.com/wordpress/wp-content/uploads/ipc-sm-782a_amendment_1_and_2.pdf), generated with kicad-footprint-generator")
 		(tags "resistor")
-		(property "Reference" "1kR1"
+		(property "Reference" "1k"
 			(at 0 1.65 90)
 			(layer "B.SilkS")
@@
 		(descr "Resistor SMD 0805 (2012 Metric), square (rectangular) end terminal, IPC-7351 nominal, (Body size source: IPC-SM-782 page 72, https://www.pcb-3d.com/wordpress/wp-content/uploads/ipc-sm-782a_amendment_1_and_2.pdf), generated with kicad-footprint-generator")
 		(tags "resistor")
-		(property "Reference" "100kR1"
+		(property "Reference" "100k"
 			(at 0 1.65 90)
 			(layer "B.SilkS")
